File: Hardware/VehicleControlUnit/Motor_Comms.kicad_sch (KiCad schematic)
At the start: 47 parts

Commit message: VCU more like diddle-u, mika time
Parts:
- removed Q?: NMOS, symbol Simulation_SPICE:NMOS
- added Q3: IRLML2030TRPBF, symbol Simulation_SPICE:NMOS
- Q4: renamed from Q?; value NMOS -> IRLML2030TRPBF; P/N (none) -> IRLML2030TRPBF
- gave numbers to parts that had none: 45
Connections:
- net PWR_MODE_IN: now also Q3.1 (D)
- net PWR_MODE_OUT: now also Q3.3 (S)
- net PwrMode_Gate: now also Q3.2 (G)
- net SPI_CLK: no longer IC6.3 (INA)
- net SPI_CS: no longer IC6.5 (INC)
- net SPI_MOSI: no longer IC6.4 (INB)
- new net DAC_CLK: IC6.3 (INA)
- new net DAC_CS: IC6.5 (INC)
- new net DAC_MOSI: IC6.4 (INB)
Other:
- moved on the sheet: C35, C37, D17, D18, IC4, IC5, IC6, JP2, PS1, Q4, R35, R36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

Commit message: mika changes
Parts:
- removed TP7: TestPoint, symbol Connector:TestPoint
- added C35, C36: 2.2uF, symbol Device:C
- renumbered C35 to C37, C36 to C38, C37 to C39
Connections:
- net SPI_CLK is gone; now on net DAC_CLK: TP24.1
- net SPI_CS is gone; now on net DAC_CS: TP26.1
- net SPI_MOSI is gone; now on net DAC_MOSI: TP25.1
- net +3.3V: now also C35.2
- net GND: now also C36.2
- net GND_ISO: now also C36.1
- net at L2.1, PS1.4 (+VOUT): now also C35.1
Other:
- moved on the sheet: C39, L2, PS1, TP10, TP11, TP12, TP13, TP17, TP18, TP19, TP20, TP25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

Commit message: need to add foot prints and start layout
Parts:
- added JP5: SolderJumper_2_Open, symbol Jumper:SolderJumper_2_Open
- C36: renamed from C35; now not fitted
- C37: renamed from C36; now not fitted
- renumbered C39 to C35, C37 to C38, C38 to C39, TP11 to TP10, TP12 to TP11, TP13 to TP12, TP14 to TP13, TP15 to TP14, TP16 to TP15, TP17 to TP16, TP18 to TP17, TP19 to TP18, TP20 to TP19, TP21 to TP20, TP22 to TP21, TP23 to TP22, TP24 to TP23, TP25 to TP24, TP26 to TP25, TP8 to TP7, TP9 to TP8, TP10 to TP9
Connections:
- net +3.3V: now also C35.1, L2.2, JP5.1 (A); no longer C36.2, PS1.2 (+VIN)
- net +3.3V_ISO: now also C36.1, PS1.4 (+VOUT); no longer C35.1, L2.2
- net GND: now also C35.2
- net GND_ISO: no longer C35.2
- new net: C36.2, JP5.2 (B), L2.1, PS1.2 (+VIN)
Other:
- moved on the sheet: C35, L2, PS1

Commit message: ughhhhhhhhhhhhhhhhhhh VCU will lokwey explode and propell the car
Parts:
- removed TP10, TP11, TP12, TP13, TP14, TP15, TP16, TP17, TP18, TP19, TP20, TP21, TP22, TP23, TP24, TP25, TP5, TP6, TP7, TP8, TP9: TestPoint, symbol Connector:TestPoint
- added J10: Debug_PinHeader, symbol Connector_Generic:Conn_02x11_Counter_Clockwise
- added R48: 5.1k, symbol Device:R
- added R49: 9.1k, symbol Device:R
- renumbered R35 to R40, R36 to R41, R37 to R42, R38 to R43, R39 to R44, R40 to R45, R41 to R46, R42 to R47
Connections:
- net +3.3V: now also J10.1 (Pin_1)
- net +3.3V_ISO: now also J10.22 (Pin_22)
- net Accel_DAC: now also J10.4 (Pin_4)
- net Brake_DAC: now also J10.3 (Pin_3)
- net CAN_RX: now also J10.10 (Pin_10)
- net CAN_TX: now also J10.11 (Pin_11)
- net DAC_CLK: now also J10.15 (Pin_15)
- net DAC_CS: now also J10.13 (Pin_13)
- net DAC_MOSI: now also J10.14 (Pin_14)
- net FWD_EN: now also J10.6 (Pin_6)
- net F/R_Mode: now also J10.19 (Pin_19)
- net GND: now also J10.2 (Pin_2), R49.2
- net GND_ISO: now also J10.21 (Pin_21)
- net LDAC: now also J10.5 (Pin_5)
- net Mtr_CANH: now also J10.9 (Pin_9)
- net Mtr_CANL: now also J10.8 (Pin_8)
- net PWR_MODE_EN: now also J10.7 (Pin_7)
- net PwrMode_Gate: now also J10.20 (Pin_20)
- net SPI_CLK_ISO: now also J10.16 (Pin_16)
- net SPI_CS_ISO: now also J10.17 (Pin_17)
- net SPI_MOSI_ISO: now also J10.18 (Pin_18)
- new net Pulse_ADC: R48.1, R49.1
- new net Pulse_RAW: R48.2
- no-connect marks 10 -> 11
Other:
- note added: "R1"
- note added: "R2"
- note added: "RPM Pulse Step Down"

Commit message: need to update design blocks
Connections:
- net F/R_Mode: no longer IC5.13 (OUTB), Q4.2 (G), R47.2
- net GND: no longer U4.7 (Vss)
- net GND_ISO: now also U4.7 (Vss)
- new net F/R_Mode_Gate: IC5.13 (OUTB), Q4.2 (G), R47.2
Other:
- note added: "Pin Header will be finalized at layout"
- moved on the sheet: J10
