File: Hardware/VehicleControlUnit/Motor_Comms.kicad_sch (KiCad schematic)
At the start: 31 parts, among them IC4 ISO1042QDWRQ1, IC5 ISO7741DWR, IC6 ISO7741DWR, J10 Debug_PinHeader, Q3 IRLML2030TRPBF, Q4 IRLML2030TRPBF, U4 MCP4822

Commit message: pre layout
Parts:
- C40: renamed from C34; footprint (none) -> Capacitor_SMD:C_0603_1608Metric_Pad1.08x0.95mm_HandSolder
- C41: renamed from C35; footprint (none) -> Capacitor_SMD:C_0603_1608Metric_Pad1.08x0.95mm_HandSolder
- C42: renamed from C36; footprint (none) -> Capacitor_SMD:C_0603_1608Metric_Pad1.08x0.95mm_HandSolder
- C43: renamed from C37; footprint (none) -> Capacitor_SMD:C_0603_1608Metric_Pad1.08x0.95mm_HandSolder
- C44: renamed from C38; footprint (none) -> Capacitor_SMD:C_0603_1608Metric_Pad1.08x0.95mm_HandSolder
- C45: renamed from C39; footprint (none) -> Capacitor_SMD:C_0603_1608Metric_Pad1.08x0.95mm_HandSolder
- D17, D18: footprint (none) -> LED_SMD:LED_0603_1608Metric
- IC4: footprint SOIC127P1030X265-16N -> ISO1042QDWRQ1:ISO1042QDWRQ1
- IC5, IC6: footprint SOIC127P1030X265-16N -> ISO7741DWR:ISO7741DWR
- JP2, JP4: footprint (none) -> Jumper:SolderJumper-2_P1.3mm_Bridged2Bar_RoundedPad1.0x1.5mm
- JP3, JP5: footprint (none) -> Jumper:SolderJumper-2_P1.3mm_Open_RoundedPad1.0x1.5mm
- L2: footprint (none) -> 10uH_inducto:WE-MAIA_2512
- PS1: footprint RM-3.33.3S:CONV_RM-3.33.3S -> RM-3.33.3SHP:RM-3.33.3SHP
- Q3, Q4: footprint (none) -> IRLML2030TRPBF:IRLML2030TRPBF
- R41: renamed from R40; footprint (none) -> Resistor_SMD:R_0603_1608Metric_Pad0.98x0.95mm_HandSolder
- R42: renamed from R41; footprint (none) -> Resistor_SMD:R_0603_1608Metric_Pad0.98x0.95mm_HandSolder
- R43: renamed from R42; footprint (none) -> Resistor_SMD:R_0603_1608Metric_Pad0.98x0.95mm_HandSolder
- R44: renamed from R43; footprint (none) -> Resistor_SMD:R_0603_1608Metric_Pad0.98x0.95mm_HandSolder
- R45: renamed from R44; footprint (none) -> Resistor_SMD:R_0603_1608Metric_Pad0.98x0.95mm_HandSolder
- R46: renamed from R45; footprint (none) -> Resistor_SMD:R_0603_1608Metric_Pad0.98x0.95mm_HandSolder
- R47: renamed from R46; footprint (none) -> Resistor_SMD:R_0603_1608Metric_Pad0.98x0.95mm_HandSolder
- R48: renamed from R47; footprint (none) -> Resistor_SMD:R_0603_1608Metric_Pad0.98x0.95mm_HandSolder
- R49: renamed from R48; footprint (none) -> Resistor_SMD:R_0603_1608Metric_Pad0.98x0.95mm_HandSolder
- R50: renamed from R49; footprint (none) -> Resistor_SMD:R_0603_1608Metric_Pad0.98x0.95mm_HandSolder
- U5: renamed from U4; footprint (none) -> MCP4822T-E_SN:MCP4822T-E_SN
- renumbered J10 to J11

Commit message: stoopid lck files
Parts:
- removed PS1: RM-3.33.3S, RM-3.33.3SHP:RM-3.33.3SHP, symbol RM-3.33.3S:RM-3.33.3S
- added PS1: ROE-3.305S, ROE-3.305S:CONV_ROE-3.305S, symbol ROE-3.305S:ROE-3.305S
- J11: footprint (none) -> Connector_PinHeader_1.00mm:PinHeader_2x11_P1.00mm_Vertical
Connections:
- net +3.3V: no longer C44.2, C45.2, U5.1 (Vdd)
- net +3.3V_ISO: now also C44.2, C45.2, U5.1 (Vdd), PS1.4 (+VOUT)
- net GND: now also PS1.1 (-VIN); no longer C44.1, C45.1
- net GND_ISO: now also C44.1, C45.1, PS1.3 (-VOUT)
- net at C42.2, JP5.2 (B), L2.1: now also PS1.2 (+VIN)
