File: Hardware/VehicleControlUnit/CarCAN.kicad_sch (KiCad schematic)
At the start: 9 parts, among them IC1 TCAN3413DR

Commit message: VCU more like diddle-u, mika time
Parts:
- renumbered C5 to C14, C6 to C15, C7 to C16, C8 to C17, D8 to D4, IC1 to IC2, JP2 to JP1, R23 to R10, R22 to R9
Changed lines of the file:
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@@
 	(text "CAN Transceiver\n"
 		(exclude_from_sim no)
-		(at 69.596 49.784 0)
+		(at 69.85 49.53 0)
 		(effects
 			(font
@@
 	(text "Try to keep CDSOT23 near bus conn"
 		(exclude_from_sim no)
-		(at 197.866 64.008 0)
+		(at 198.12 63.5 0)
 		(effects
 			(font
@@
 	(text "CAN Protection"
 		(exclude_from_sim no)
-		(at 177.546 43.942 0)
+		(at 177.8 44.45 0)
 		(effects
 			(font
@@
 	(text "CAN Bus Termination\n"
 		(exclude_from_sim no)
-		(at 181.864 76.454 0)
+		(at 181.61 76.2 0)
 		(effects
 			(font
@@
 		(in_pos_files yes)
 		(dnp no)
-		(property "Reference" "C6"
+		(property "Reference" "C15"
 			(at 76.2 73.66 0)
 			(show_name no)
@@
 			(project "VehicleControlUnit"
 				(path "/e864fac9-3897-46c9-9101-6d5488c6cd3a/252635d1-b56c-4964-8f6e-39efe20521e2"
-					(reference "C6")
+					(reference "C15")
 					(unit 1)
 				)
@@
 		(in_pos_files yes)
 		(dnp no)
-		(property "Reference" "C8"
+		(property "Reference" "C17"
 			(at 194.564 88.646 0)
 			(show_name no)
@@
 			(project "VehicleControlUnit"
 				(path "/e864fac9-3897-46c9-9101-6d5488c6cd3a/252635d1-b56c-4964-8f6e-39efe20521e2"
-					(reference "C8")
+					(reference "C17")
 					(unit 1)
 				)
@@
 		(dnp no)
 		(fields_autoplaced yes)
-		(property "Reference" "JP2"
+		(property "Reference" "JP1"
 			(at 215.9 78.74 0)
 			(show_name no)
@@
 			(project "VehicleControlUnit"
 				(path "/e864fac9-3897-46c9-9101-6d5488c6cd3a/252635d1-b56c-4964-8f6e-39efe20521e2"
-					(reference "JP2")
+					(reference "JP1")
 					(unit 1)
 				)
@@
 		(in_pos_files yes)
 		(dnp no)
-		(property "Reference" "C7"
+		(property "Reference" "C16"
 			(at 88.138 73.66 0)
 			(show_name no)
@@
 			(project "VehicleControlUnit"
 				(path "/e864fac9-3897-46c9-9101-6d5488c6cd3a/252635d1-b56c-4964-8f6e-39efe20521e2"
-					(reference "C7")
+					(reference "C16")
 					(unit 1)
 				)
@@
 		(in_pos_files yes)
 		(dnp no)
-		(property "Reference" "C5"
+		(property "Reference" "C14"
 			(at 65.278 73.66 0)
 			(show_name no)
@@
 			(project "VehicleControlUnit"
 				(path "/e864fac9-3897-46c9-9101-6d5488c6cd3a/252635d1-b56c-4964-8f6e-39efe20521e2"
-					(reference "C5")
+					(reference "C14")
 					(unit 1)
 				)
@@
 		(in_pos_files yes)
 		(dnp no)
-		(property "Reference" "R23"
+		(property "Reference" "R10"
 			(at 201.93 80.01 90)
 			(show_name no)
@@
 			(project "VehicleControlUnit"
 				(path "/e864fac9-3897-46c9-9101-6d5488c6cd3a/252635d1-b56c-4964-8f6e-39efe20521e2"
-					(reference "R23")
+					(reference "R10")
 					(unit 1)
 				)
@@
 		(dnp no)
 		(fields_autoplaced yes)
-		(property "Reference" "D8"
+		(property "Reference" "D4"
 			(at 196.85 46.99 0)
 			(show_name no)
@@
 			(project "VehicleControlUnit"
 				(path "/e864fac9-3897-46c9-9101-6d5488c6cd3a/252635d1-b56c-4964-8f6e-39efe20521e2"
-					(reference "D8")
+					(reference "D4")
 					(unit 1)
 				)
@@
 		(dnp no)
 		(fields_autoplaced yes)
-		(property "Reference" "IC1"
+		(property "Reference" "IC2"
 			(at 128.27 63.5 0)
 			(show_name no)
@@
 			(project "VehicleControlUnit"
 				(path "/e864fac9-3897-46c9-9101-6d5488c6cd3a/252635d1-b56c-4964-8f6e-39efe20521e2"
-					(reference "IC1")
+					(reference "IC2")
 					(unit 1)
 				)
@@
 		(in_pos_files yes)
 		(dnp no)
-		(property "Reference" "R22"
+		(property "Reference" "R9"
 			(at 176.53 80.01 90)
 			(show_name no)
@@
 			(project "VehicleControlUnit"
 				(path "/e864fac9-3897-46c9-9101-6d5488c6cd3a/252635d1-b56c-4964-8f6e-39efe20521e2"
-					(reference "R22")
-					(unit 1)
-				)
+					(reference "R9")
+					(unit 1)
+				)

Commit message: ughhhhhhhhhhhhhhhhhhh VCU will lokwey explode and propell the car
Parts:
- renumbered R9 to R13, R10 to R14
Changed lines of the file:
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@@
 		(in_pos_files yes)
 		(dnp no)
-		(property "Reference" "R10"
+		(property "Reference" "R14"
 			(at 201.93 80.01 90)
 			(show_name no)
@@
 			(project "VehicleControlUnit"
 				(path "/e864fac9-3897-46c9-9101-6d5488c6cd3a/252635d1-b56c-4964-8f6e-39efe20521e2"
-					(reference "R10")
+					(reference "R14")
 					(unit 1)
 				)
@@
 		(in_pos_files yes)
 		(dnp no)
-		(property "Reference" "R9"
+		(property "Reference" "R13"
 			(at 176.53 80.01 90)
 			(show_name no)
@@
 			(project "VehicleControlUnit"
 				(path "/e864fac9-3897-46c9-9101-6d5488c6cd3a/252635d1-b56c-4964-8f6e-39efe20521e2"
-					(reference "R9")
-					(unit 1)
-				)
+					(reference "R13")
+					(unit 1)
+				)

Commit message: pre layout
Parts:
- renumbered C14 to C20, C15 to C21, C16 to C22, C17 to C23, R13 to R14, R14 to R15
Changed lines of the file:
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@@
 		(in_pos_files yes)
 		(dnp no)
-		(property "Reference" "C15"
+		(property "Reference" "C21"
 			(at 76.2 73.66 0)
 			(show_name no)
@@
 			(project "VehicleControlUnit"
 				(path "/e864fac9-3897-46c9-9101-6d5488c6cd3a/252635d1-b56c-4964-8f6e-39efe20521e2"
-					(reference "C15")
+					(reference "C21")
 					(unit 1)
 				)
@@
 		(in_pos_files yes)
 		(dnp no)
-		(property "Reference" "C17"
+		(property "Reference" "C23"
 			(at 194.564 88.646 0)
 			(show_name no)
@@
 			(project "VehicleControlUnit"
 				(path "/e864fac9-3897-46c9-9101-6d5488c6cd3a/252635d1-b56c-4964-8f6e-39efe20521e2"
-					(reference "C17")
+					(reference "C23")
 					(unit 1)
 				)
@@
 		(in_pos_files yes)
 		(dnp no)
-		(property "Reference" "C16"
+		(property "Reference" "C22"
 			(at 88.138 73.66 0)
 			(show_name no)
@@
 			(project "VehicleControlUnit"
 				(path "/e864fac9-3897-46c9-9101-6d5488c6cd3a/252635d1-b56c-4964-8f6e-39efe20521e2"
-					(reference "C16")
+					(reference "C22")
 					(unit 1)
 				)
@@
 		(in_pos_files yes)
 		(dnp no)
-		(property "Reference" "C14"
+		(property "Reference" "C20"
 			(at 65.278 73.66 0)
 			(show_name no)
@@
 			(project "VehicleControlUnit"
 				(path "/e864fac9-3897-46c9-9101-6d5488c6cd3a/252635d1-b56c-4964-8f6e-39efe20521e2"
-					(reference "C14")
+					(reference "C20")
 					(unit 1)
 				)
@@
 		(in_pos_files yes)
 		(dnp no)
-		(property "Reference" "R14"
+		(property "Reference" "R15"
 			(at 201.93 80.01 90)
 			(show_name no)
@@
 			(project "VehicleControlUnit"
 				(path "/e864fac9-3897-46c9-9101-6d5488c6cd3a/252635d1-b56c-4964-8f6e-39efe20521e2"
-					(reference "R14")
+					(reference "R15")
 					(unit 1)
 				)
@@
 		(in_pos_files yes)
 		(dnp no)
-		(property "Reference" "R13"
+		(property "Reference" "R14"
 			(at 176.53 80.01 90)
 			(show_name no)
@@
 			(project "VehicleControlUnit"
 				(path "/e864fac9-3897-46c9-9101-6d5488c6cd3a/252635d1-b56c-4964-8f6e-39efe20521e2"
-					(reference "R13")
-					(unit 1)
-				)
+					(reference "R14")
+					(unit 1)
+				)
