File: Hardware/VehicleControlUnit/PowerProtection.kicad_sch (KiCad schematic)
At the start: 18 parts

Commit message: VCU more like diddle-u, mika time
Parts:
- gave numbers to parts that had none: 18
Changed lines of the file:
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@@
 		(in_pos_files yes)
 		(dnp no)
-		(property "Reference" "C?"
+		(property "Reference" "C13"
 			(at 125.984 89.154 90)
 			(show_name no)
@@
 			(project "VehicleControlUnit"
 				(path "/e864fac9-3897-46c9-9101-6d5488c6cd3a/f16a8bc3-f058-4d27-badd-0afc148d009e/19de6bb4-fd37-45ed-ab7a-91a6842df4d8"
-					(reference "C?")
+					(reference "C13")
 					(unit 1)
 				)
@@
 		(in_pos_files yes)
 		(dnp no)
-		(property "Reference" "D?"
+		(property "Reference" "D3"
 			(at 40.64 82.296 0)
 			(show_name no)
@@
 			(project "VehicleControlUnit"
 				(path "/e864fac9-3897-46c9-9101-6d5488c6cd3a/f16a8bc3-f058-4d27-badd-0afc148d009e/19de6bb4-fd37-45ed-ab7a-91a6842df4d8"
-					(reference "D?")
+					(reference "D3")
 					(unit 1)
 				)
@@
 		(dnp no)
 		(fields_autoplaced yes)
-		(property "Reference" "C?"
+		(property "Reference" "C9"
 			(at 57.785 80.0099 0)
 			(show_name no)
@@
 			(project "VehicleControlUnit"
 				(path "/e864fac9-3897-46c9-9101-6d5488c6cd3a/f16a8bc3-f058-4d27-badd-0afc148d009e/19de6bb4-fd37-45ed-ab7a-91a6842df4d8"
-					(reference "C?")
+					(reference "C9")
 					(unit 1)
 				)
@@
 		(in_pos_files yes)
 		(dnp no)
-		(property "Reference" "D?"
+		(property "Reference" "D2"
 			(at 22.606 49.276 0)
 			(show_name no)
@@
 			(project "VehicleControlUnit"
 				(path "/e864fac9-3897-46c9-9101-6d5488c6cd3a/f16a8bc3-f058-4d27-badd-0afc148d009e/19de6bb4-fd37-45ed-ab7a-91a6842df4d8"
-					(reference "D?")
+					(reference "D2")
 					(unit 1)
 				)
@@
 		(dnp no)
 		(fields_autoplaced yes)
-		(property "Reference" "R?"
+		(property "Reference" "R3"
 			(at 45.72 60.9599 0)
 			(show_name no)
@@
 			(project "VehicleControlUnit"
 				(path "/e864fac9-3897-46c9-9101-6d5488c6cd3a/f16a8bc3-f058-4d27-badd-0afc148d009e/19de6bb4-fd37-45ed-ab7a-91a6842df4d8"
-					(reference "R?")
+					(reference "R3")
 					(unit 1)
 				)
@@
 		(in_pos_files yes)
 		(dnp no)
-		(property "Reference" "R?"
+		(property "Reference" "R8"
 			(at 137.668 90.17 90)
 			(show_name no)
@@
 			(project "VehicleControlUnit"
 				(path "/e864fac9-3897-46c9-9101-6d5488c6cd3a/f16a8bc3-f058-4d27-badd-0afc148d009e/19de6bb4-fd37-45ed-ab7a-91a6842df4d8"
-					(reference "R?")
+					(reference "R8")
 					(unit 1)
 				)
@@
 		(in_pos_files yes)
 		(dnp no)
-		(property "Reference" "C?"
+		(property "Reference" "C7"
 			(at 38.1 49.5299 0)
 			(show_name no)
@@
 			(project "VehicleControlUnit"
 				(path "/e864fac9-3897-46c9-9101-6d5488c6cd3a/f16a8bc3-f058-4d27-badd-0afc148d009e/19de6bb4-fd37-45ed-ab7a-91a6842df4d8"
-					(reference "C?")
+					(reference "C7")
 					(unit 1)
 				)
@@
 		(in_pos_files yes)
 		(dnp no)
-		(property "Reference" "R?"
+		(property "Reference" "R4"
 			(at 67.31 54.61 90)
 			(show_name no)
@@
 			(project "VehicleControlUnit"
 				(path "/e864fac9-3897-46c9-9101-6d5488c6cd3a/f16a8bc3-f058-4d27-badd-0afc148d009e/19de6bb4-fd37-45ed-ab7a-91a6842df4d8"
-					(reference "R?")
+					(reference "R4")
 					(unit 1)
 				)
@@
 		(in_pos_files yes)
 		(dnp no)
-		(property "Reference" "C?"
+		(property "Reference" "C12"
 			(at 107.188 88.9 90)
 			(show_name no)
@@
 			(project "VehicleControlUnit"
 				(path "/e864fac9-3897-46c9-9101-6d5488c6cd3a/f16a8bc3-f058-4d27-badd-0afc148d009e/19de6bb4-fd37-45ed-ab7a-91a6842df4d8"
-					(reference "C?")
+					(reference "C12")
 					(unit 1)
 				)
@@
 		(in_pos_files yes)
 		(dnp no)
-		(property "Reference" "IC?"
+		(property "Reference" "IC1"
 			(at 75.184 73.66 0)
 			(show_name no)
@@
 			(project "VehicleControlUnit"
 				(path "/e864fac9-3897-46c9-9101-6d5488c6cd3a/f16a8bc3-f058-4d27-badd-0afc148d009e/19de6bb4-fd37-45ed-ab7a-91a6842df4d8"
-					(reference "IC?")
+					(reference "IC1")
 					(unit 1)
 				)
@@
 		(in_pos_files yes)
 		(dnp no)
-		(property "Reference" "Q?"
+		(property "Reference" "Q1"
 			(at 52.578 38.862 90)
 			(show_name no)
@@
 			(project "VehicleControlUnit"
 				(path "/e864fac9-3897-46c9-9101-6d5488c6cd3a/f16a8bc3-f058-4d27-badd-0afc148d009e/19de6bb4-fd37-45ed-ab7a-91a6842df4d8"
-					(reference "Q?")
+					(reference "Q1")
 					(unit 1)
 				)
@@
 		(in_pos_files yes)
 		(dnp no)
-		(property "Reference" "C?"
+		(property "Reference" "C10"
 			(at 54.864 62.23 0)
 			(show_name no)
@@
 			(project "VehicleControlUnit"
 				(path "/e864fac9-3897-46c9-9101-6d5488c6cd3a/f16a8bc3-f058-4d27-badd-0afc148d009e/19de6bb4-fd37-45ed-ab7a-91a6842df4d8"
-					(reference "C?")
+					(reference "C10")
 					(unit 1)
 				)
@@
 		(in_pos_files yes)
 		(dnp no)
-		(property "Reference" "C?"
+		(property "Reference" "C11"
 			(at 112.395 49.5299 0)
 			(show_name no)
@@
 			(project "VehicleControlUnit"
 				(path "/e864fac9-3897-46c9-9101-6d5488c6cd3a/f16a8bc3-f058-4d27-badd-0afc148d009e/19de6bb4-fd37-45ed-ab7a-91a6842df4d8"
-					(reference "C?")
+					(reference "C11")
 					(unit 1)
 				)
@@
 		(in_pos_files yes)
 		(dnp no)
-		(property "Reference" "Q?"
+		(property "Reference" "Q2"
 			(at 100.584 38.608 90)
 			(show_name no)
@@
 			(project "VehicleControlUnit"
 				(path "/e864fac9-3897-46c9-9101-6d5488c6cd3a/f16a8bc3-f058-4d27-badd-0afc148d009e/19de6bb4-fd37-45ed-ab7a-91a6842df4d8"
-					(reference "Q?")
+					(reference "Q2")
 					(unit 1)
 				)
@@
 		(in_pos_files yes)
 		(dnp no)
-		(property "Reference" "R?"
+		(property "Reference" "R6"
 			(at 118.618 90.424 90)
 			(show_name no)
@@
 			(project "VehicleControlUnit"
 				(path "/e864fac9-3897-46c9-9101-6d5488c6cd3a/f16a8bc3-f058-4d27-badd-0afc148d009e/19de6bb4-fd37-45ed-ab7a-91a6842df4d8"
-					(reference "R?")
+					(reference "R6")
 					(unit 1)
 				)
@@
 		(in_pos_files yes)
 		(dnp no)
-		(property "Reference" "C?"
+		(property "Reference" "C8"
 			(at 31.75 82.5499 0)
 			(show_name no)
@@
 			(project "VehicleControlUnit"
 				(path "/e864fac9-3897-46c9-9101-6d5488c6cd3a/f16a8bc3-f058-4d27-badd-0afc148d009e/19de6bb4-fd37-45ed-ab7a-91a6842df4d8"
-					(reference "C?")
+					(reference "C8")
 					(unit 1)
 				)
@@
 		(in_pos_files yes)
 		(dnp no)
-		(property "Reference" "R?"
+		(property "Reference" "R5"
 			(at 118.11 78.74 90)
 			(show_name no)
@@
 			(project "VehicleControlUnit"
 				(path "/e864fac9-3897-46c9-9101-6d5488c6cd3a/f16a8bc3-f058-4d27-badd-0afc148d009e/19de6bb4-fd37-45ed-ab7a-91a6842df4d8"
-					(reference "R?")
+					(reference "R5")
 					(unit 1)
 				)
@@
 		(in_pos_files yes)
 		(dnp no)
-		(property "Reference" "R?"
+		(property "Reference" "R7"
 			(at 137.16 77.47 90)
 			(show_name no)
@@
 			(project "VehicleControlUnit"
 				(path "/e864fac9-3897-46c9-9101-6d5488c6cd3a/f16a8bc3-f058-4d27-badd-0afc148d009e/19de6bb4-fd37-45ed-ab7a-91a6842df4d8"
-					(reference "R?")
+					(reference "R7")
 					(unit 1)
 				)

Commit message: ughhhhhhhhhhhhhhhhhhh VCU will lokwey explode and propell the car
Parts:
- renumbered R6 to R10, R7 to R11, R8 to R12, R3 to R7, R4 to R8, R5 to R9
Changed lines of the file:
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@@
 		(dnp no)
 		(fields_autoplaced yes)
-		(property "Reference" "R3"
+		(property "Reference" "R7"
 			(at 45.72 60.9599 0)
 			(show_name no)
@@
 			(project "VehicleControlUnit"
 				(path "/e864fac9-3897-46c9-9101-6d5488c6cd3a/f16a8bc3-f058-4d27-badd-0afc148d009e/19de6bb4-fd37-45ed-ab7a-91a6842df4d8"
-					(reference "R3")
+					(reference "R7")
 					(unit 1)
 				)
@@
 		(in_pos_files yes)
 		(dnp no)
-		(property "Reference" "R8"
+		(property "Reference" "R12"
 			(at 137.668 90.17 90)
 			(show_name no)
@@
 			(project "VehicleControlUnit"
 				(path "/e864fac9-3897-46c9-9101-6d5488c6cd3a/f16a8bc3-f058-4d27-badd-0afc148d009e/19de6bb4-fd37-45ed-ab7a-91a6842df4d8"
-					(reference "R8")
+					(reference "R12")
 					(unit 1)
 				)
@@
 		(in_pos_files yes)
 		(dnp no)
-		(property "Reference" "R4"
+		(property "Reference" "R8"
 			(at 67.31 54.61 90)
 			(show_name no)
@@
 			(project "VehicleControlUnit"
 				(path "/e864fac9-3897-46c9-9101-6d5488c6cd3a/f16a8bc3-f058-4d27-badd-0afc148d009e/19de6bb4-fd37-45ed-ab7a-91a6842df4d8"
-					(reference "R4")
+					(reference "R8")
 					(unit 1)
 				)
@@
 		(in_pos_files yes)
 		(dnp no)
-		(property "Reference" "R6"
+		(property "Reference" "R10"
 			(at 118.618 90.424 90)
 			(show_name no)
@@
 			(project "VehicleControlUnit"
 				(path "/e864fac9-3897-46c9-9101-6d5488c6cd3a/f16a8bc3-f058-4d27-badd-0afc148d009e/19de6bb4-fd37-45ed-ab7a-91a6842df4d8"
-					(reference "R6")
+					(reference "R10")
 					(unit 1)
 				)
@@
 		(in_pos_files yes)
 		(dnp no)
-		(property "Reference" "R5"
+		(property "Reference" "R9"
 			(at 118.11 78.74 90)
 			(show_name no)
@@
 			(project "VehicleControlUnit"
 				(path "/e864fac9-3897-46c9-9101-6d5488c6cd3a/f16a8bc3-f058-4d27-badd-0afc148d009e/19de6bb4-fd37-45ed-ab7a-91a6842df4d8"
-					(reference "R5")
+					(reference "R9")
 					(unit 1)
 				)
@@
 		(in_pos_files yes)
 		(dnp no)
-		(property "Reference" "R7"
+		(property "Reference" "R11"
 			(at 137.16 77.47 90)
 			(show_name no)
@@
 			(project "VehicleControlUnit"
 				(path "/e864fac9-3897-46c9-9101-6d5488c6cd3a/f16a8bc3-f058-4d27-badd-0afc148d009e/19de6bb4-fd37-45ed-ab7a-91a6842df4d8"
-					(reference "R7")
+					(reference "R11")
 					(unit 1)
 				)

Commit message: pre layout
Parts:
- removed C12, C13: 0.1u, Capacitor_SMD:C_0603_1608Metric_Pad1.08x0.95mm_HandSolder, symbol Device:C
- added C6, C7: 0.1u, Capacitor_SMD:C_0603_1608Metric_Pad1.08x0.95mm_HandSolder, symbol Device:C
- C1: renamed from C7; LCSC P/N C14663 -> C1591; P/N MLASH168SB7104KTNA01 -> CL10B104KB8NNNC
- C2: renamed from C8; LCSC P/N C15849 -> C559769; P/N MLASU168SB5105KTNA01 -> CC0603KRX7R9BB105
- C3: renamed from C9; LCSC P/N C344195 -> C107083; Mouser Part Number 963-MSASU168SB7224KT -> (none); P/N MSASU168SB7224KTNB25 -> CC0603KRX7R9BB224
- C4: renamed from C10; LCSC C57112 -> (none); LCSC P/N MSASH168SB5103KTNA01 -> C100042; P/N (none) -> CC0603KRX7R9BB103
- C5: renamed from C11; P/N GRM21BR61H106KE43K -> GRM21BR61H106KE43L
- D2: renamed from D3; LCSC P/N (none) -> C183490; P/N (none) -> SMAF4758A
- R10: renamed from R12; LCSC P/N C2090646 -> C843918; P/N CRCW0603137KFKEA -> CRCW060315K8FKEA
- R5: renamed from R7; Mouser Part Number 71-CRCW060310K0FKEI -> (none); P/N CRCW060310K0FKEI -> 0603WAF1002T5E
- R6: renamed from R8; LCSC P/N C844927 -> C2074308; Mouser Part Number 594-MCT06030C2003FP5 -> 594-MCT06030C3309FP5; P/N CRCW060333R0FKEA -> MCT06030C3309FP500
- R7: renamed from R9; LCSC P/N C2090661 -> C25803; P/N CRCW0603221KFKEA -> 0603WAF1003T5E
- R8: renamed from R10; LCSC P/N C25804 -> C862286; P/N CRCW060310K0FKEI -> RT0603BRE077K32L
- R9: renamed from R11; LCSC P/N C25804 -> C25803; P/N CRCW060310K0FKEI -> 0603WAF1003T5E
- renumbered D2 to D1
Connections:
- net EN/UVLO: now also C7.1
- net GND: now also C6.2, C7.2
- net OV: now also C6.1
