File: Hardware/VehicleControlUnit/Power_Mux.kicad_sch (KiCad schematic)
At the start: 6 parts, among them U1 TPS2117DRLR

Commit message: VCU more like diddle-u, mika time
Parts:
- renumbered C1 to C38, C2 to C39, C3 to C40, C4 to C41, R1 to R46, U1 to U5
Changed lines of the file:
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@@
 		(in_pos_files yes)
 		(dnp no)
-		(property "Reference" "C4"
+		(property "Reference" "C41"
 			(at 91.8972 57.2516 0)
 			(show_name no)
@@
 			(project "VehicleControlUnit"
 				(path "/e864fac9-3897-46c9-9101-6d5488c6cd3a/f16a8bc3-f058-4d27-badd-0afc148d009e/59ba047e-cc6c-42e3-939f-b33701d25ed0"
-					(reference "C4")
+					(reference "C41")
 					(unit 1)
 				)
@@
 		(in_pos_files yes)
 		(dnp no)
-		(property "Reference" "R1"
+		(property "Reference" "R46"
 			(at 78.994 67.564 0)
 			(show_name no)
@@
 			(project "VehicleControlUnit"
 				(path "/e864fac9-3897-46c9-9101-6d5488c6cd3a/f16a8bc3-f058-4d27-badd-0afc148d009e/59ba047e-cc6c-42e3-939f-b33701d25ed0"
-					(reference "R1")
+					(reference "R46")
 					(unit 1)
 				)
@@
 		(in_pos_files yes)
 		(dnp no)
-		(property "Reference" "C1"
+		(property "Reference" "C38"
 			(at 24.5872 44.5516 0)
 			(show_name no)
@@
 			(project "VehicleControlUnit"
 				(path "/e864fac9-3897-46c9-9101-6d5488c6cd3a/f16a8bc3-f058-4d27-badd-0afc148d009e/59ba047e-cc6c-42e3-939f-b33701d25ed0"
-					(reference "C1")
+					(reference "C38")
 					(unit 1)
 				)
@@
 		(dnp no)
 		(fields_autoplaced yes)
-		(property "Reference" "U1"
+		(property "Reference" "U5"
 			(at 60.96 44.45 0)
 			(show_name no)
@@
 			(project "VehicleControlUnit"
 				(path "/e864fac9-3897-46c9-9101-6d5488c6cd3a/f16a8bc3-f058-4d27-badd-0afc148d009e/59ba047e-cc6c-42e3-939f-b33701d25ed0"
-					(reference "U1")
+					(reference "U5")
 					(unit 1)
 				)
@@
 		(in_pos_files yes)
 		(dnp no)
-		(property "Reference" "C3"
+		(property "Reference" "C40"
 			(at 42.3672 67.4116 0)
 			(show_name no)
@@
 			(project "VehicleControlUnit"
 				(path "/e864fac9-3897-46c9-9101-6d5488c6cd3a/f16a8bc3-f058-4d27-badd-0afc148d009e/59ba047e-cc6c-42e3-939f-b33701d25ed0"
-					(reference "C3")
+					(reference "C40")
 					(unit 1)
 				)
@@
 		(in_pos_files yes)
 		(dnp no)
-		(property "Reference" "C2"
+		(property "Reference" "C39"
 			(at 38.5572 44.5516 0)
 			(show_name no)
@@
 			(project "VehicleControlUnit"
 				(path "/e864fac9-3897-46c9-9101-6d5488c6cd3a/f16a8bc3-f058-4d27-badd-0afc148d009e/59ba047e-cc6c-42e3-939f-b33701d25ed0"
-					(reference "C2")
-					(unit 1)
-				)
+					(reference "C39")
+					(unit 1)
+				)

Commit message: mika changes
Parts:
- renumbered C38 to C40, C39 to C41, C40 to C42, C41 to C43
Changed lines of the file:
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@@
 		(in_pos_files yes)
 		(dnp no)
-		(property "Reference" "C41"
+		(property "Reference" "C43"
 			(at 91.8972 57.2516 0)
 			(show_name no)
@@
 			(project "VehicleControlUnit"
 				(path "/e864fac9-3897-46c9-9101-6d5488c6cd3a/f16a8bc3-f058-4d27-badd-0afc148d009e/59ba047e-cc6c-42e3-939f-b33701d25ed0"
-					(reference "C41")
+					(reference "C43")
 					(unit 1)
 				)
@@
 		(in_pos_files yes)
 		(dnp no)
-		(property "Reference" "C38"
+		(property "Reference" "C40"
 			(at 24.5872 44.5516 0)
 			(show_name no)
@@
 			(project "VehicleControlUnit"
 				(path "/e864fac9-3897-46c9-9101-6d5488c6cd3a/f16a8bc3-f058-4d27-badd-0afc148d009e/59ba047e-cc6c-42e3-939f-b33701d25ed0"
-					(reference "C38")
+					(reference "C40")
 					(unit 1)
 				)
@@
 		(in_pos_files yes)
 		(dnp no)
-		(property "Reference" "C40"
+		(property "Reference" "C42"
 			(at 42.3672 67.4116 0)
 			(show_name no)
@@
 			(project "VehicleControlUnit"
 				(path "/e864fac9-3897-46c9-9101-6d5488c6cd3a/f16a8bc3-f058-4d27-badd-0afc148d009e/59ba047e-cc6c-42e3-939f-b33701d25ed0"
-					(reference "C40")
+					(reference "C42")
 					(unit 1)
 				)
@@
 		(in_pos_files yes)
 		(dnp no)
-		(property "Reference" "C39"
+		(property "Reference" "C41"
 			(at 38.5572 44.5516 0)
 			(show_name no)
@@
 			(project "VehicleControlUnit"
 				(path "/e864fac9-3897-46c9-9101-6d5488c6cd3a/f16a8bc3-f058-4d27-badd-0afc148d009e/59ba047e-cc6c-42e3-939f-b33701d25ed0"
-					(reference "C39")
-					(unit 1)
-				)
+					(reference "C41")
+					(unit 1)
+				)

Commit message: ughhhhhhhhhhhhhhhhhhh VCU will lokwey explode and propell the car
Parts:
- renumbered R46 to R53
Changed lines of the file:
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@@
 		(in_pos_files yes)
 		(dnp no)
-		(property "Reference" "R46"
+		(property "Reference" "R53"
 			(at 78.994 67.564 0)
 			(show_name no)
@@
 			(project "VehicleControlUnit"
 				(path "/e864fac9-3897-46c9-9101-6d5488c6cd3a/f16a8bc3-f058-4d27-badd-0afc148d009e/59ba047e-cc6c-42e3-939f-b33701d25ed0"
-					(reference "R46")
+					(reference "R53")
 					(unit 1)
 				)

Commit message: pre layout
Parts:
- renumbered C40 to C14, C41 to C15, C42 to C16, C43 to C17, R53 to R13, U5 to U2
Changed lines of the file:
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@@
 		(in_pos_files yes)
 		(dnp no)
-		(property "Reference" "C43"
+		(property "Reference" "C17"
 			(at 91.8972 57.2516 0)
 			(show_name no)
@@
 			)
 			(project "VehicleControlUnit"
-				(path "/e864fac9-3897-46c9-9101-6d5488c6cd3a/f16a8bc3-f058-4d27-badd-0afc148d009e/59ba047e-cc6c-42e3-939f-b33701d25ed0"
-					(reference "C43")
+				(path "/e864fac9-3897-46c9-9101-6d5488c6cd3a/f16a8bc3-f058-4d27-badd-0afc148d009e/d4cd4986-72cf-4091-9d22-3ed3db5e35c5"
+					(reference "C17")
 					(unit 1)
 				)
@@
 		(in_pos_files yes)
 		(dnp no)
-		(property "Reference" "R53"
+		(property "Reference" "R13"
 			(at 78.994 67.564 0)
 			(show_name no)
@@
 			)
 			(project "VehicleControlUnit"
-				(path "/e864fac9-3897-46c9-9101-6d5488c6cd3a/f16a8bc3-f058-4d27-badd-0afc148d009e/59ba047e-cc6c-42e3-939f-b33701d25ed0"
-					(reference "R53")
+				(path "/e864fac9-3897-46c9-9101-6d5488c6cd3a/f16a8bc3-f058-4d27-badd-0afc148d009e/d4cd4986-72cf-4091-9d22-3ed3db5e35c5"
+					(reference "R13")
 					(unit 1)
 				)
@@
 		(in_pos_files yes)
 		(dnp no)
-		(property "Reference" "C40"
+		(property "Reference" "C14"
 			(at 24.5872 44.5516 0)
 			(show_name no)
@@
 			)
 			(project "VehicleControlUnit"
-				(path "/e864fac9-3897-46c9-9101-6d5488c6cd3a/f16a8bc3-f058-4d27-badd-0afc148d009e/59ba047e-cc6c-42e3-939f-b33701d25ed0"
-					(reference "C40")
+				(path "/e864fac9-3897-46c9-9101-6d5488c6cd3a/f16a8bc3-f058-4d27-badd-0afc148d009e/d4cd4986-72cf-4091-9d22-3ed3db5e35c5"
+					(reference "C14")
 					(unit 1)
 				)
@@
 		(dnp no)
 		(fields_autoplaced yes)
-		(property "Reference" "U5"
+		(property "Reference" "U2"
 			(at 60.96 44.45 0)
 			(show_name no)
@@
 			)
 			(project "VehicleControlUnit"
-				(path "/e864fac9-3897-46c9-9101-6d5488c6cd3a/f16a8bc3-f058-4d27-badd-0afc148d009e/59ba047e-cc6c-42e3-939f-b33701d25ed0"
-					(reference "U5")
+				(path "/e864fac9-3897-46c9-9101-6d5488c6cd3a/f16a8bc3-f058-4d27-badd-0afc148d009e/d4cd4986-72cf-4091-9d22-3ed3db5e35c5"
+					(reference "U2")
 					(unit 1)
 				)
@@
 		(in_pos_files yes)
 		(dnp no)
-		(property "Reference" "C42"
+		(property "Reference" "C16"
 			(at 42.3672 67.4116 0)
 			(show_name no)
@@
 			)
 			(project "VehicleControlUnit"
-				(path "/e864fac9-3897-46c9-9101-6d5488c6cd3a/f16a8bc3-f058-4d27-badd-0afc148d009e/59ba047e-cc6c-42e3-939f-b33701d25ed0"
-					(reference "C42")
+				(path "/e864fac9-3897-46c9-9101-6d5488c6cd3a/f16a8bc3-f058-4d27-badd-0afc148d009e/d4cd4986-72cf-4091-9d22-3ed3db5e35c5"
+					(reference "C16")
 					(unit 1)
 				)
@@
 		(in_pos_files yes)
 		(dnp no)
-		(property "Reference" "C41"
+		(property "Reference" "C15"
 			(at 38.5572 44.5516 0)
 			(show_name no)
@@
 			)
 			(project "VehicleControlUnit"
-				(path "/e864fac9-3897-46c9-9101-6d5488c6cd3a/f16a8bc3-f058-4d27-badd-0afc148d009e/59ba047e-cc6c-42e3-939f-b33701d25ed0"
-					(reference "C41")
-					(unit 1)
-				)
+				(path "/e864fac9-3897-46c9-9101-6d5488c6cd3a/f16a8bc3-f058-4d27-badd-0afc148d009e/d4cd4986-72cf-4091-9d22-3ed3db5e35c5"
+					(reference "C15")
+					(unit 1)
+				)
