File: Hardware/VehicleControlUnit/SD_Card.kicad_sch (KiCad schematic)
At the start: 4 parts

Commit message: VCU more like diddle-u, mika time
Parts:
- gave numbers to parts that had none: 4
Connections:
- net SPI_CLK renamed SD_CLK
- net SPI_CS renamed SD_CS
- net SPI_DET renamed DET
- net SPI_MISO renamed SD_MISO
- net SPI_MOSI renamed SD_MOSI
Other:
- moved on the sheet: CR1, J7, R26, R27

Commit message: ughhhhhhhhhhhhhhhhhhh VCU will lokwey explode and propell the car
Parts:
- renumbered J7 to J9, R26 to R31, R27 to R32
Changed lines of the file:
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@@
 		(in_pos_files yes)
 		(dnp no)
-		(property "Reference" "R27"
+		(property "Reference" "R32"
 			(at 128.27 72.39 90)
 			(show_name no)
@@
 			(project "VehicleControlUnit"
 				(path "/e864fac9-3897-46c9-9101-6d5488c6cd3a/b0b52d73-b085-4624-9871-af1c22d24972"
-					(reference "R27")
+					(reference "R32")
 					(unit 1)
 				)
@@
 		(in_pos_files yes)
 		(dnp no)
-		(property "Reference" "R26"
+		(property "Reference" "R31"
 			(at 125.73 82.55 90)
 			(show_name no)
@@
 			(project "VehicleControlUnit"
 				(path "/e864fac9-3897-46c9-9101-6d5488c6cd3a/b0b52d73-b085-4624-9871-af1c22d24972"
-					(reference "R26")
+					(reference "R31")
 					(unit 1)
 				)
@@
 		(dnp no)
 		(fields_autoplaced yes)
-		(property "Reference" "J7"
+		(property "Reference" "J9"
 			(at 155.575 43.434 0)
 			(show_name no)
@@
 			(project "VehicleControlUnit"
 				(path "/e864fac9-3897-46c9-9101-6d5488c6cd3a/b0b52d73-b085-4624-9871-af1c22d24972"
-					(reference "J7")
+					(reference "J9")
 					(unit 1)
 				)

Commit message: pre layout
Parts:
- CR1: footprint SOT26_DIO -> LHRS_ICs:D5V0P4UR6SO-7
- J10: renamed from J9; footprint (none) -> Connector_Card:microSD_HC_Hirose_DM3AT-SF-PEJM5
- R32: renamed from R31; footprint (none) -> Resistor_SMD:R_0603_1608Metric_Pad0.98x0.95mm_HandSolder
- R33: renamed from R32; footprint (none) -> Resistor_SMD:R_0603_1608Metric_Pad0.98x0.95mm_HandSolder
Changed lines of the file:
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@@
 		(in_pos_files yes)
 		(dnp no)
-		(property "Reference" "R32"
+		(property "Reference" "R33"
 			(at 128.27 72.39 90)
 			(show_name no)
@@
 			)
 		)
-		(property "Footprint" ""
+		(property "Footprint" "Resistor_SMD:R_0603_1608Metric_Pad0.98x0.95mm_HandSolder"
 			(at 128.27 68.072 90)
 			(hide yes)
@@
 			(project "VehicleControlUnit"
 				(path "/e864fac9-3897-46c9-9101-6d5488c6cd3a/b0b52d73-b085-4624-9871-af1c22d24972"
-					(reference "R32")
+					(reference "R33")
 					(unit 1)
 				)
@@
 		(in_pos_files yes)
 		(dnp no)
-		(property "Reference" "R31"
+		(property "Reference" "R32"
 			(at 125.73 82.55 90)
 			(show_name no)
@@
 			)
 		)
-		(property "Footprint" ""
+		(property "Footprint" "Resistor_SMD:R_0603_1608Metric_Pad0.98x0.95mm_HandSolder"
 			(at 125.73 78.232 90)
 			(hide yes)
@@
 			(project "VehicleControlUnit"
 				(path "/e864fac9-3897-46c9-9101-6d5488c6cd3a/b0b52d73-b085-4624-9871-af1c22d24972"
-					(reference "R31")
+					(reference "R32")
 					(unit 1)
 				)
@@
 		(dnp no)
 		(fields_autoplaced yes)
-		(property "Reference" "J9"
+		(property "Reference" "J10"
 			(at 155.575 43.434 0)
 			(show_name no)
@@
 			)
 		)
-		(property "Footprint" ""
+		(property "Footprint" "Connector_Card:microSD_HC_Hirose_DM3AT-SF-PEJM5"
 			(at 207.01 46.99 0)
 			(hide yes)
@@
 			(project "VehicleControlUnit"
 				(path "/e864fac9-3897-46c9-9101-6d5488c6cd3a/b0b52d73-b085-4624-9871-af1c22d24972"
-					(reference "J9")
+					(reference "J10")
 					(unit 1)
 				)
@@
 			)
 		)
-		(property "Footprint" "SOT26_DIO"
+		(property "Footprint" "LHRS_ICs:D5V0P4UR6SO-7"
 			(at 40.64 53.34 0)
 			(hide yes)
