File: Hardware/VehicleControlUnit/motor_fans.kicad_sch (KiCad schematic)
At the start: 12 parts

Commit message: VCU more like diddle-u, mika time
Parts:
- gave numbers to parts that had none: 12
Connections:
- net FAN_SDA is gone; now on net FAN_SCL: IC3.1 (SMDATA), R28.2
- net ALERT: now also IC3.11 (CLK), R34.2
- net FAN_SCL: now also IC3.4 (ADDR_SEL), R30.2
Other:
- moved on the sheet: D15, IC3, R28, R29, R30, R31, R32, R33, R34

Commit message: mika changes
Connections:
- net ALERT: no longer IC3.11 (CLK), R34.2
- net FAN_SCL: no longer IC3.1 (SMDATA), IC3.4 (ADDR_SEL), R28.2, R30.2
- new net: IC3.11 (CLK), R34.2
- new net: IC3.4 (ADDR_SEL), R30.2
- new net FAN_SDA: IC3.1 (SMDATA), R28.2
Other:
- moved on the sheet: R28, R29, R30, R33, R34
Changed lines of the file:
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@@
 	)
 	(junction
-		(at 66.04 40.64)
+		(at 66.04 38.1)
 		(diameter 0)
 		(color 0 0 0 0)
 	)
 	(junction
-		(at 71.12 49.53)
+		(at 66.04 49.53)
 		(diameter 0)
 		(color 0 0 0 0)
@@
 	)
 	(junction
-		(at 113.03 49.53)
-		(diameter 0)
-		(color 0 0 0 0)
-	)
-	(junction
 		(at 109.22 77.47)
 		(diameter 0)
@@
 	)
 	(junction
-		(at 69.85 40.64)
-		(diameter 0)
-		(color 0 0 0 0)
-	)
-	(junction
-		(at 71.12 52.07)
+		(at 113.03 49.53)
 		(diameter 0)
 		(color 0 0 0 0)
 	)
 	(junction
-		(at 66.04 49.53)
+		(at 69.85 38.1)
 		(diameter 0)
 		(color 0 0 0 0)
 	)
 	(junction
-		(at 91.44 76.2)
+		(at 71.12 52.07)
 		(diameter 0)
 		(color 0 0 0 0)
@@
 	)
 	(junction
-		(at 74.93 49.53)
-		(diameter 0)
-		(color 0 0 0 0)
-	)
-	(junction
-		(at 116.84 49.53)
+		(at 91.44 76.2)
 		(diameter 0)
 		(color 0 0 0 0)
 	)
 	(junction
-		(at 116.84 40.64)
+		(at 116.84 38.1)
 		(diameter 0)
 		(color 0 0 0 0)
@@
 	(wire
 		(pts
-			(xy 71.12 41.91) (xy 69.85 40.64)
+			(xy 71.12 39.37) (xy 69.85 38.1)
 		)
 		(stroke
@@
 	(wire
 		(pts
-			(xy 71.12 49.53) (xy 74.93 49.53)
+			(xy 66.04 49.53) (xy 76.2 49.53)
 		)
 		(stroke
@@
 	(wire
 		(pts
-			(xy 63.5 40.64) (xy 66.04 40.64)
+			(xy 66.04 46.99) (xy 66.04 49.53)
+		)
+		(stroke
+			(width 0)
+			(type default)
+		)
+	)
+	(wire
+		(pts
+			(xy 63.5 38.1) (xy 66.04 38.1)
 		)
 		(stroke
@@
 	(wire
 		(pts
-			(xy 116.84 49.53) (xy 118.11 49.53)
+			(xy 113.03 49.53) (xy 118.11 49.53)
 		)
 		(stroke
@@
 	(wire
 		(pts
-			(xy 74.93 49.53) (xy 76.2 49.53)
-		)
-		(stroke
-			(width 0)
-			(type default)
-		)
-	)
-	(wire
-		(pts
 			(xy 64.77 77.47) (xy 67.31 77.47)
 		)
@@
 	(wire
 		(pts
-			(xy 69.85 40.64) (xy 73.66 40.64)
+			(xy 69.85 38.1) (xy 73.66 38.1)
 		)
 		(stroke
@@
 	(wire
 		(pts
-			(xy 114.3 40.64) (xy 116.84 40.64)
+			(xy 114.3 38.1) (xy 116.84 38.1)
 		)
 		(stroke
@@
 	(wire
 		(pts
-			(xy 113.03 49.53) (xy 116.84 49.53)
-		)
-		(stroke
-			(width 0)
-			(type default)
-		)
-	)
-	(wire
-		(pts
 			(xy 93.98 78.74) (xy 93.98 74.93)
 		)
@@
 	(wire
 		(pts
-			(xy 113.03 41.91) (xy 114.3 40.64)
+			(xy 113.03 39.37) (xy 114.3 38.1)
 		)
 		(stroke
@@
 	(wire
 		(pts
-			(xy 74.93 49.53) (xy 74.93 55.88)
-		)
-		(stroke
-			(width 0)
-			(type default)
-		)
-	)
-	(wire
-		(pts
-			(xy 66.04 40.64) (xy 69.85 40.64)
+			(xy 74.93 46.99) (xy 74.93 55.88)
 		)
 		(stroke
@@
 	(wire
 		(pts
-			(xy 66.04 49.53) (xy 71.12 49.53)
+			(xy 66.04 38.1) (xy 69.85 38.1)
 		)
 		(stroke
@@
 	(wire
 		(pts
-			(xy 116.84 40.64) (xy 119.38 40.64)
+			(xy 116.84 38.1) (xy 119.38 38.1)
 		)
 		(stroke
@@
 	(wire
 		(pts
-			(xy 66.04 40.64) (xy 66.04 41.91)
+			(xy 66.04 38.1) (xy 66.04 39.37)
 		)
 		(stroke
@@
 	(wire
 		(pts
-			(xy 116.84 49.53) (xy 116.84 50.8)
+			(xy 116.84 46.99) (xy 116.84 50.8)
 		)
 		(stroke
@@
 	(wire
 		(pts
-			(xy 71.12 49.53) (xy 71.12 52.07)
+			(xy 71.12 46.99) (xy 71.12 52.07)
 		)
 		(stroke
@@
 	(wire
 		(pts
-			(xy 74.93 41.91) (xy 73.66 40.64)
+			(xy 74.93 39.37) (xy 73.66 38.1)
 		)
 		(stroke
@@
 	(wire
 		(pts
-			(xy 116.84 40.64) (xy 116.84 41.91)
+			(xy 116.84 38.1) (xy 116.84 39.37)
 		)
 		(stroke
@@
 	(wire
 		(pts
+			(xy 113.03 46.99) (xy 113.03 49.53)
+		)
+		(stroke
+			(width 0)
+			(type default)
+		)
+	)
+	(wire
+		(pts
 			(xy 111.76 49.53) (xy 113.03 49.53)
 		)
@@
 	(hierarchical_label "+3.3V"
 		(shape input)
-		(at 63.5 40.64 180)
+		(at 63.5 38.1 180)
 		(effects
 			(font
@@
 	(hierarchical_label "+3.3V"
 		(shape input)
-		(at 119.38 40.64 0)
+		(at 119.38 38.1 0)
 		(effects
 			(font
@@
 	(symbol
 		(lib_id "Device:R")
-		(at 66.04 45.72 0)
+		(at 66.04 43.18 0)
 		(unit 1)
 		(body_style 1)
@@
 		(dnp no)
 		(property "Reference" "R28"
-			(at 62.992 45.72 0)
+			(at 62.992 43.18 0)
 			(show_name no)
 			(do_not_autoplace no)
@@
 		)
 		(property "Value" "10k"
-			(at 66.04 45.72 90)
+			(at 66.04 43.18 90)
 			(show_name no)
 			(do_not_autoplace no)
@@
 		)
 		(property "Footprint" ""
-			(at 64.262 45.72 90)
+			(at 64.262 43.18 90)
 			(hide yes)
 			(show_name no)
@@
 		)
 		(property "Datasheet" ""
-			(at 66.04 45.72 0)
+			(at 66.04 43.18 0)
 			(hide yes)
 			(show_name no)
@@
 		)
 		(property "Description" "Resistor"
-			(at 66.04 45.72 0)
+			(at 66.04 43.18 0)
 			(hide yes)
 			(show_name no)
@@
 	(symbol
 		(lib_id "Device:R")
-		(at 113.03 45.72 0)
+		(at 113.03 43.18 0)
 		(unit 1)
 		(body_style 1)
@@
 		(dnp no)
 		(property "Reference" "R33"
-			(at 110.49 45.974 0)
+			(at 110.49 43.434 90)
 			(show_name no)
 			(do_not_autoplace no)
@@
 		)
 		(property "Value" "10k"
-			(at 113.03 45.72 90)
+			(at 113.03 43.18 90)
 			(show_name no)
 			(do_not_autoplace no)
@@
 		)
 		(property "Footprint" ""
-			(at 111.252 45.72 90)
+			(at 111.252 43.18 90)
 			(hide yes)
 			(show_name no)
@@
 		)
 		(property "Datasheet" ""
-			(at 113.03 45.72 0)
+			(at 113.03 43.18 0)
 			(hide yes)
 			(show_name no)
@@
 		)
 		(property "Description" "Resistor"
-			(at 113.03 45.72 0)
+			(at 113.03 43.18 0)
 			(hide yes)
 			(show_name no)
@@
 	(symbol
 		(lib_id "Device:R")
-		(at 116.84 45.72 0)
+		(at 116.84 43.18 0)
 		(unit 1)
 		(body_style 1)
@@
 		(dnp no)
 		(property "Reference" "R34"
-			(at 119.888 45.974 0)
+			(at 119.888 43.434 90)
 			(show_name no)
 			(do_not_autoplace no)
@@
 		)
 		(property "Value" "33k"
-			(at 116.84 45.72 90)
+			(at 116.84 43.18 90)
 			(show_name no)
 			(do_not_autoplace no)
@@
 		)
 		(property "Footprint" ""
-			(at 115.062 45.72 90)
+			(at 115.062 43.18 90)
 			(hide yes)
 			(show_name no)
@@
 		)
 		(property "Datasheet" ""
-			(at 116.84 45.72 0)
+			(at 116.84 43.18 0)
 			(hide yes)
 			(show_name no)
@@
 		)
 		(property "Description" "Resistor"
-			(at 116.84 45.72 0)
+			(at 116.84 43.18 0)
 			(hide yes)
 			(show_name no)
@@
 	(symbol
 		(lib_id "Device:R")
-		(at 71.12 45.72 0)
+		(at 71.12 43.18 0)
 		(unit 1)
 		(body_style 1)
@@
 		(dnp no)
 		(property "Reference" "R29"
-			(at 68.58 45.72 90)
+			(at 68.58 43.18 90)
 			(show_name no)
 			(do_not_autoplace no)
@@
 		)
 		(property "Value" "10k"
-			(at 71.12 45.72 90)
+			(at 71.12 43.18 90)
 			(show_name no)
 			(do_not_autoplace no)
@@
 		)
 		(property "Footprint" ""
-			(at 69.342 45.72 90)
+			(at 69.342 43.18 90)
 			(hide yes)
 			(show_name no)
@@
 		)
 		(property "Datasheet" ""
-			(at 71.12 45.72 0)
+			(at 71.12 43.18 0)
 			(hide yes)
 			(show_name no)
@@
 		)
 		(property "Description" "Resistor"
-			(at 71.12 45.72 0)
+			(at 71.12 43.18 0)
 			(hide yes)
 			(show_name no)
@@
 	(symbol
 		(lib_id "Device:R")
-		(at 74.93 45.72 0)
+		(at 74.93 43.18 0)
 		(unit 1)
 		(body_style 1)
@@
 		(dnp no)
 		(property "Reference" "R30"
-			(at 77.724 45.212 0)
+			(at 77.724 42.672 0)
 			(show_name no)
 			(do_not_autoplace no)
@@
 		)
 		(property "Value" "33k"
-			(at 74.93 45.72 90)
+			(at 74.93 43.18 90)
 			(show_name no)
 			(do_not_autoplace no)
@@
 		)
 		(property "Footprint" ""
-			(at 73.152 45.72 90)
+			(at 73.152 43.18 90)
 			(hide yes)
 			(show_name no)
@@
 		)
 		(property "Datasheet" ""
-			(at 74.93 45.72 0)
+			(at 74.93 43.18 0)
 			(hide yes)
 			(show_name no)
@@
 		)
 		(property "Description" "Resistor"
-			(at 74.93 45.72 0)
+			(at 74.93 43.18 0)
 			(hide yes)
 			(show_name no)

Commit message: ughhhhhhhhhhhhhhhhhhh VCU will lokwey explode and propell the car
Parts:
- renumbered D16 to D15, D15 to D16, R28 to R33, R29 to R34, R30 to R35, R31 to R36, R32 to R37, R33 to R38, R34 to R39
Other:
- moved on the sheet: D15, D16

Commit message: need to update design blocks
Connections:
- net +12V renamed +12V_Fan
Other:
- moved on the sheet: D15, D16
Changed lines of the file:
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@@
 	(paper "A5")
 	(rectangle
-		(start 48.514 69.85)
-		(end 76.708 93.472)
+		(start 46.99 69.85)
+		(end 80.01 93.472)
 		(stroke
 			(width 0)
@@
 	(text "Flyback Diodes"
 		(exclude_from_sim no)
-		(at 55.88 68.58 0)
+		(at 53.34 68.58 0)
 		(effects
 			(font
@@
 	)
 	(junction
-		(at 62.23 88.9)
+		(at 52.07 64.77)
 		(diameter 0)
 		(color 0 0 0 0)
 	)
 	(junction
-		(at 52.07 64.77)
+		(at 57.15 54.61)
 		(diameter 0)
 		(color 0 0 0 0)
 	)
 	(junction
-		(at 57.15 54.61)
+		(at 109.22 77.47)
 		(diameter 0)
 		(color 0 0 0 0)
 	)
 	(junction
-		(at 62.23 76.2)
+		(at 113.03 49.53)
 		(diameter 0)
 		(color 0 0 0 0)
 	)
 	(junction
-		(at 109.22 77.47)
+		(at 69.85 38.1)
 		(diameter 0)
 		(color 0 0 0 0)
 	)
 	(junction
-		(at 113.03 49.53)
+		(at 71.12 52.07)
 		(diameter 0)
 		(color 0 0 0 0)
 	)
 	(junction
-		(at 69.85 38.1)
+		(at 59.69 81.28)
 		(diameter 0)
 		(color 0 0 0 0)
 	)
 	(junction
-		(at 71.12 52.07)
+		(at 72.39 81.28)
 		(diameter 0)
 		(color 0 0 0 0)
@@
 	(wire
 		(pts
-			(xy 62.23 88.9) (xy 66.04 88.9)
+			(xy 60.96 86.36) (xy 59.69 85.09)
 		)
 		(stroke
@@
 	(wire
 		(pts
-			(xy 57.15 77.47) (xy 58.42 76.2)
+			(xy 71.12 39.37) (xy 69.85 38.1)
 		)
 		(stroke
@@
 	(wire
 		(pts
-			(xy 71.12 39.37) (xy 69.85 38.1)
+			(xy 86.36 30.48) (xy 87.63 30.48)
 		)
 		(stroke
@@
 	(wire
 		(pts
-			(xy 86.36 30.48) (xy 87.63 30.48)
+			(xy 59.69 81.28) (xy 59.69 77.47)
 		)
 		(stroke
@@
 	(wire
 		(pts
-			(xy 57.15 78.74) (xy 57.15 77.47)
+			(xy 62.23 86.36) (xy 60.96 86.36)
 		)
 		(stroke
@@
 	(wire
 		(pts
+			(xy 58.42 81.28) (xy 59.69 81.28)
+		)
+		(stroke
+			(width 0)
+			(type default)
+		)
+	)
+	(wire
+		(pts
 			(xy 115.57 52.07) (xy 116.84 50.8)
 		)
@@
 	(wire
 		(pts
-			(xy 67.31 78.74) (xy 67.31 77.47)
+			(xy 62.23 76.2) (xy 60.96 76.2)
 		)
 		(stroke
@@
 	(wire
 		(pts
+			(xy 72.39 81.28) (xy 73.66 81.28)
+		)
+		(stroke
+			(width 0)
+			(type default)
+		)
+	)
+	(wire
+		(pts
 			(xy 52.07 54.61) (xy 57.15 54.61)
 		)
@@
 	(wire
 		(pts
-			(xy 58.42 76.2) (xy 62.23 76.2)
+			(xy 59.69 85.09) (xy 59.69 81.28)
 		)
 		(stroke
@@
 	(wire
 		(pts
-			(xy 57.15 86.36) (xy 57.15 87.63)
+			(xy 69.85 86.36) (xy 71.12 86.36)
 		)
 		(stroke
@@
 	(wire
 		(pts
-			(xy 67.31 86.36) (xy 67.31 87.63)
+			(xy 69.85 76.2) (xy 71.12 76.2)
 		)
 		(stroke
@@
 	(wire
 		(pts
-			(xy 67.31 77.47) (xy 66.04 76.2)
+			(xy 60.96 76.2) (xy 59.69 77.47)
 		)
 		(stroke
@@
 	(wire
 		(pts
-			(xy 57.15 87.63) (xy 58.42 88.9)
+			(xy 71.12 86.36) (xy 72.39 85.09)
 		)
 		(stroke
@@
 	(wire
 		(pts
-			(xy 57.15 55.88) (xy 57.15 54.61)
+			(xy 72.39 85.09) (xy 72.39 81.28)
 		)
 		(stroke
@@
 	(wire
 		(pts
-			(xy 62.23 88.9) (xy 62.23 91.44)
+			(xy 72.39 81.28) (xy 72.39 77.47)
 		)
 		(stroke
@@
 	(wire
 		(pts
-			(xy 116.84 46.99) (xy 116.84 50.8)
+			(xy 57.15 55.88) (xy 57.15 54.61)
 		)
 		(stroke
@@
 	(wire
 		(pts
-			(xy 71.12 52.07) (xy 76.2 52.07)
+			(xy 116.84 46.99) (xy 116.84 50.8)
 		)
 		(stroke
@@
 	(wire
 		(pts
-			(xy 71.12 46.99) (xy 71.12 52.07)
+			(xy 71.12 52.07) (xy 76.2 52.07)
 		)
 		(stroke
@@
 	(wire
 		(pts
-			(xy 66.04 88.9) (xy 67.31 87.63)
+			(xy 71.12 46.99) (xy 71.12 52.07)
 		)
 		(stroke
@@
 	(wire
 		(pts
-			(xy 74.93 39.37) (xy 73.66 38.1)
+			(xy 72.39 77.47) (xy 71.12 76.2)
 		)
 		(stroke
@@
 	(wire
 		(pts
-			(xy 74.93 55.88) (xy 76.2 57.15)
+			(xy 74.93 39.37) (xy 73.66 38.1)
 		)
 		(stroke
@@
 	(wire
 		(pts
-			(xy 116.84 38.1) (xy 116.84 39.37)
+			(xy 74.93 55.88) (xy 76.2 57.15)
 		)
 		(stroke
@@
 	(wire
 		(pts
-			(xy 63.5 49.53) (xy 66.04 49.53)
+			(xy 116.84 38.1) (xy 116.84 39.37)
 		)
 		(stroke
@@
 	(wire
 		(pts
-			(xy 113.03 46.99) (xy 113.03 49.53)
+			(xy 63.5 49.53) (xy 66.04 49.53)
 		)
 		(stroke
@@
 	(wire
 		(pts
-			(xy 58.42 88.9) (xy 62.23 88.9)
+			(xy 113.03 46.99) (xy 113.03 49.53)
 		)
 		(stroke
@@
 		)
 	)
-	(wire
-		(pts
-			(xy 62.23 76.2) (xy 66.04 76.2)
-		)
-		(stroke
-			(width 0)
-			(type default)
-		)
-	)
 	(image
 		(at 149.86 67.056)
@@
 		)
 	)
+	(hierarchical_label "+12V_Fan"
+		(shape input)
+		(at 58.42 81.28 180)
+		(effects
+			(font
+				(size 1.27 1.27)
+			)
+			(justify right)
+		)
+	)
 	(hierarchical_label "GND"
 		(shape input)
-		(at 62.23 91.44 0)
+		(at 73.66 81.28 0)
 		(effects
 			(font
@@
 	)
 	(symbol
-		(lib_id "power:+12V")
-		(at 62.23 76.2 0)
-		(mirror y)
-		(unit 1)
-		(body_style 1)
-		(exclude_from_sim no)
-		(in_bom yes)
-		(on_board yes)
-		(in_pos_files yes)
-		(dnp no)
-		(property "Reference" "#PWR026"
-			(at 62.23 80.01 0)
-			(hide yes)
-			(show_name no)
-			(do_not_autoplace no)
-			(effects
-				(font
-					(size 1.27 1.27)
-				)
-			)
-		)
-		(property "Value" "+12V"
-			(at 62.23 72.39 0)
-			(show_name no)
-			(do_not_autoplace no)
-			(effects
-				(font
-					(size 1.27 1.27)
-				)
-			)
-		)
-		(property "Footprint" ""
-			(at 62.23 76.2 0)
-			(hide yes)
-			(show_name no)
-			(do_not_autoplace no)
-			(effects
-				(font
-					(size 1.27 1.27)
-				)
-			)
-		)
-		(property "Datasheet" ""
-			(at 62.23 76.2 0)
-			(hide yes)
-			(show_name no)
-			(do_not_autoplace no)
-			(effects
-				(font
-					(size 1.27 1.27)
-				)
-			)
-		)
-		(property "Description" "Power symbol creates a global label with name \"+12V\""
-			(at 62.23 76.2 0)
-			(hide yes)
-			(show_name no)
-			(do_not_autoplace no)
-			(effects
-				(font
-					(size 1.27 1.27)
-				)
-			)
-		)
-		(pin "1"
-		)
-		(instances
-			(project "VehicleControlUnit"
-				(path "/e864fac9-3897-46c9-9101-6d5488c6cd3a/76867641-26a4-43d1-a64a-9a6eb791f3f7"
-					(reference "#PWR026")
-					(unit 1)
-				)
-			)
-		)
-	)
-	(symbol
 		(lib_id "Device:R")
 		(at 113.03 43.18 0)
@@
 	(symbol
 		(lib_id "Device:D_Schottky")
-		(at 57.15 82.55 90)
+		(at 66.04 86.36 0)
 		(mirror x)
 		(unit 1)
@@
 		(dnp no)
 		(property "Reference" "D15"
-			(at 60.198 81.534 0)
+			(at 65.024 83.312 0)
 			(show_name no)
 			(do_not_autoplace no)
@@
 		)
 		(property "Value" "D_Schottky"
-			(at 54.102 77.47 0)
+			(at 60.96 89.408 0)
 			(show_name no)
 			(do_not_autoplace no)
@@
 		)
 		(property "Footprint" ""
-			(at 57.15 82.55 0)
+			(at 66.04 86.36 0)
 			(hide yes)
 			(show_name no)
@@
 		)
 		(property "Datasheet" ""
-			(at 57.15 82.55 0)
+			(at 66.04 86.36 0)
 			(hide yes)
 			(show_name no)
@@
 		)
 		(property "Description" "Schottky diode"
-			(at 57.15 82.55 0)
+			(at 66.04 86.36 0)
 			(hide yes)
 			(show_name no)
@@
 		(dnp no)
 		(property "Reference" "C32"
-			(at 49.022 57.15 0)
+			(at 46.99 57.15 0)
 			(show_name no)
 			(do_not_autoplace no)
@@
 	(symbol
 		(lib_id "Device:D_Schottky")
-		(at 67.31 82.55 90)
+		(at 66.04 76.2 0)
 		(mirror x)
 		(unit 1)
@@
 		(dnp no)
 		(property "Reference" "D16"
-			(at 70.358 81.534 0)
+			(at 65.024 73.152 0)
 			(show_name no)
 			(do_not_autoplace no)
@@
 		)
 		(property "Value" "D_Schottky"
-			(at 64.262 77.47 0)
+			(at 60.96 79.248 0)
 			(show_name no)
 			(do_not_autoplace no)
@@
 		)
 		(property "Footprint" ""
-			(at 67.31 82.55 0)
+			(at 66.04 76.2 0)
 			(hide yes)
 			(show_name no)
@@
 		)
 		(property "Datasheet" ""
-			(at 67.31 82.55 0)
+			(at 66.04 76.2 0)
 			(hide yes)
 			(show_name no)
@@
 		)
 		(property "Description" "Schottky diode"
-			(at 67.31 82.55 0)
+			(at 66.04 76.2 0)
 			(hide yes)
 			(show_name no)

Commit message: pre layout
Parts:
- C38: renamed from C32; footprint (none) -> Capacitor_SMD:C_0603_1608Metric_Pad1.08x0.95mm_HandSolder
- C39: renamed from C33; footprint (none) -> Capacitor_SMD:C_0603_1608Metric_Pad1.08x0.95mm_HandSolder
- D15: renamed from D16; footprint (none) -> VSSAF522-M3_H:SODFL5226X100N
- D16: renamed from D15; footprint (none) -> VSSAF522-M3_H:SODFL5226X100N
- IC3: footprint QFN65P400X400X90-17N-D -> EMC2305-1-AP-TR:EMC2305-1-AP-TR
- R34: renamed from R33; footprint (none) -> Resistor_SMD:R_0603_1608Metric_Pad0.98x0.95mm_HandSolder
- R35: renamed from R34; footprint (none) -> Resistor_SMD:R_0603_1608Metric_Pad0.98x0.95mm_HandSolder
- R36: renamed from R35; footprint (none) -> Resistor_SMD:R_0603_1608Metric_Pad0.98x0.95mm_HandSolder
- R37: renamed from R36; footprint (none) -> Resistor_SMD:R_0603_1608Metric_Pad0.98x0.95mm_HandSolder
- R38: renamed from R37; footprint (none) -> Resistor_SMD:R_0603_1608Metric_Pad0.98x0.95mm_HandSolder
- R39: renamed from R38; footprint (none) -> Resistor_SMD:R_0603_1608Metric_Pad0.98x0.95mm_HandSolder
- R40: renamed from R39; footprint (none) -> Resistor_SMD:R_0603_1608Metric_Pad0.98x0.95mm_HandSolder
Changed lines of the file:
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@@
 		(in_pos_files yes)
 		(dnp no)
-		(property "Reference" "R33"
+		(property "Reference" "R34"
 			(at 62.992 43.18 0)
 			(show_name no)
@@
 			)
 		)
-		(property "Footprint" ""
+		(property "Footprint" "Resistor_SMD:R_0603_1608Metric_Pad0.98x0.95mm_HandSolder"
 			(at 64.262 43.18 90)
 			(hide yes)
@@
 			(project "VehicleControlUnit"
 				(path "/e864fac9-3897-46c9-9101-6d5488c6cd3a/76867641-26a4-43d1-a64a-9a6eb791f3f7"
-					(reference "R33")
+					(reference "R34")
 					(unit 1)
 				)
@@
 		(in_pos_files yes)
 		(dnp no)
-		(property "Reference" "R38"
+		(property "Reference" "R39"
 			(at 110.49 43.434 90)
 			(show_name no)
@@
 			)
 		)
-		(property "Footprint" ""
+		(property "Footprint" "Resistor_SMD:R_0603_1608Metric_Pad0.98x0.95mm_HandSolder"
 			(at 111.252 43.18 90)
 			(hide yes)
@@
 			(project "VehicleControlUnit"
 				(path "/e864fac9-3897-46c9-9101-6d5488c6cd3a/76867641-26a4-43d1-a64a-9a6eb791f3f7"
-					(reference "R38")
+					(reference "R39")
 					(unit 1)
 				)
@@
 		(in_pos_files yes)
 		(dnp no)
-		(property "Reference" "D15"
+		(property "Reference" "D16"
 			(at 65.024 83.312 0)
 			(show_name no)
@@
 			)
 		)
-		(property "Footprint" ""
+		(property "Footprint" "VSSAF522-M3_H:SODFL5226X100N"
 			(at 66.04 86.36 0)
 			(hide yes)
@@
 			(project "VehicleControlUnit"
 				(path "/e864fac9-3897-46c9-9101-6d5488c6cd3a/76867641-26a4-43d1-a64a-9a6eb791f3f7"
-					(reference "D15")
+					(reference "D16")
 					(unit 1)
 				)
@@
 		(in_pos_files yes)
 		(dnp no)
-		(property "Reference" "C33"
+		(property "Reference" "C39"
 			(at 57.912 57.15 0)
 			(show_name no)
@@
 			)
 		)
-		(property "Footprint" ""
+		(property "Footprint" "Capacitor_SMD:C_0603_1608Metric_Pad1.08x0.95mm_HandSolder"
 			(at 58.1152 63.5 0)
 			(hide yes)
@@
 			(project "VehicleControlUnit"
 				(path "/e864fac9-3897-46c9-9101-6d5488c6cd3a/76867641-26a4-43d1-a64a-9a6eb791f3f7"
-					(reference "C33")
+					(reference "C39")
 					(unit 1)
 				)
@@
 		(in_pos_files yes)
 		(dnp no)
-		(property "Reference" "R37"
+		(property "Reference" "R38"
 			(at 104.648 81.026 90)
 			(show_name no)
@@
 			)
 		)
-		(property "Footprint" ""
+		(property "Footprint" "Resistor_SMD:R_0603_1608Metric_Pad0.98x0.95mm_HandSolder"
 			(at 104.14 80.518 90)
 			(hide yes)
@@
 			(project "VehicleControlUnit"
 				(path "/e864fac9-3897-46c9-9101-6d5488c6cd3a/76867641-26a4-43d1-a64a-9a6eb791f3f7"
-					(reference "R37")
+					(reference "R38")
 					(unit 1)
 				)
@@
 			)
 		)
-		(property "Footprint" "QFN65P400X400X90-17N-D"
+		(property "Footprint" "EMC2305-1-AP-TR:EMC2305-1-AP-TR"
 			(at 107.95 134.29 0)
 			(hide yes)
@@
 		(in_pos_files yes)
 		(dnp no)
-		(property "Reference" "R39"
+		(property "Reference" "R40"
 			(at 119.888 43.434 90)
 			(show_name no)
@@
 			)
 		)
-		(property "Footprint" ""
+		(property "Footprint" "Resistor_SMD:R_0603_1608Metric_Pad0.98x0.95mm_HandSolder"
 			(at 115.062 43.18 90)
 			(hide yes)
@@
 			(project "VehicleControlUnit"
 				(path "/e864fac9-3897-46c9-9101-6d5488c6cd3a/76867641-26a4-43d1-a64a-9a6eb791f3f7"
-					(reference "R39")
+					(reference "R40")
 					(unit 1)
 				)
@@
 		(in_pos_files yes)
 		(dnp no)
-		(property "Reference" "R34"
+		(property "Reference" "R35"
 			(at 68.58 43.18 90)
 			(show_name no)
@@
 			)
 		)
-		(property "Footprint" ""
+		(property "Footprint" "Resistor_SMD:R_0603_1608Metric_Pad0.98x0.95mm_HandSolder"
 			(at 69.342 43.18 90)
 			(hide yes)
@@
 			(project "VehicleControlUnit"
 				(path "/e864fac9-3897-46c9-9101-6d5488c6cd3a/76867641-26a4-43d1-a64a-9a6eb791f3f7"
-					(reference "R34")
+					(reference "R35")
 					(unit 1)
 				)
@@
 		(in_pos_files yes)
 		(dnp no)
-		(property "Reference" "C32"
+		(property "Reference" "C38"
 			(at 46.99 57.15 0)
 			(show_name no)
@@
 			)
 		)
-		(property "Footprint" ""
+		(property "Footprint" "Capacitor_SMD:C_0603_1608Metric_Pad1.08x0.95mm_HandSolder"
 			(at 53.0352 63.5 0)
 			(hide yes)
@@
 			(project "VehicleControlUnit"
 				(path "/e864fac9-3897-46c9-9101-6d5488c6cd3a/76867641-26a4-43d1-a64a-9a6eb791f3f7"
-					(reference "C32")
+					(reference "C38")
 					(unit 1)
 				)
@@
 		(in_pos_files yes)
 		(dnp no)
-		(property "Reference" "R36"
+		(property "Reference" "R37"
 			(at 104.14 74.168 90)
 			(show_name no)
@@
 			)
 		)
-		(property "Footprint" ""
+		(property "Footprint" "Resistor_SMD:R_0603_1608Metric_Pad0.98x0.95mm_HandSolder"
 			(at 104.14 77.978 90)
 			(hide yes)
@@
 			(project "VehicleControlUnit"
 				(path "/e864fac9-3897-46c9-9101-6d5488c6cd3a/76867641-26a4-43d1-a64a-9a6eb791f3f7"
-					(reference "R36")
+					(reference "R37")
 					(unit 1)
 				)
@@
 		(in_pos_files yes)
 		(dnp no)
-		(property "Reference" "R35"
+		(property "Reference" "R36"
 			(at 77.724 42.672 0)
 			(show_name no)
@@
 			)
 		)
-		(property "Footprint" ""
+		(property "Footprint" "Resistor_SMD:R_0603_1608Metric_Pad0.98x0.95mm_HandSolder"
 			(at 73.152 43.18 90)
 			(hide yes)
@@
 			(project "VehicleControlUnit"
 				(path "/e864fac9-3897-46c9-9101-6d5488c6cd3a/76867641-26a4-43d1-a64a-9a6eb791f3f7"
-					(reference "R35")
+					(reference "R36")
 					(unit 1)
 				)
@@
 		(in_pos_files yes)
 		(dnp no)
-		(property "Reference" "D16"
+		(property "Reference" "D15"
 			(at 65.024 73.152 0)
 			(show_name no)
@@
 			)
 		)
-		(property "Footprint" ""
+		(property "Footprint" "VSSAF522-M3_H:SODFL5226X100N"
 			(at 66.04 76.2 0)
 			(hide yes)
@@
 			(project "VehicleControlUnit"
 				(path "/e864fac9-3897-46c9-9101-6d5488c6cd3a/76867641-26a4-43d1-a64a-9a6eb791f3f7"
-					(reference "D16")
-					(unit 1)
-				)
+					(reference "D15")
+					(unit 1)
+				)

Commit message: stoopid lck files
Parts:
- added TP5, TP6, TP7, TP8, TP9: TestPoint, diddle_shah:TestPoint_HEX_3mmID, symbol Connector:TestPoint
Connections:
- net ALERT: now also TP5.1
- net FAN1_PWM: now also TP6.1
- net FAN1_TACH: now also TP7.1
- net FAN_SCL: now also TP9.1
- net FAN_SDA: now also TP8.1
Other:
- moved on the sheet: D15, D16
